File: eagle_v65/Z_sim_v2.brd (EAGLE design)
At the start: 237.8 x 110.5 mm, 280 parts, among them IC1 MCP2200S, IC100 ADUM1250, IC101 LP2985, IC102 ADP7118AUJZ, IC103 ADP7182AUJZ, IC104 ADUM1250, IC105 ACSL-6210, IC106 LP2985, IC2 OPA548TH, IC3 ATmega88, IC4 OP211, IC5 MAX4820, K1 POWER, K10 TE280370, K100 G6KU-2F-Y, K101 G6KU-2F-Y, K102 G6KU-2F-Y, K11 G6KU-2F-Y, K15 G6KU-2F-Y, K16 TE280372, K19 ISP-prog, K2 PWR LED, K24 GPIO, K25 SPI bus, K26 RELAYS, K9 TE280370, Q1 12MHz, Q100 BC817-16, Q101 BC817-16, U1 LTC2631, U100 LTC2631, X1 PN61729-S, X2 Bcur, X3 Bcur, X4 Lcur, X5 Hcur, X6 Lpot, X7 Hpot, X8 Bpot, X9 Bpot

Commit message: fix: updated doc
Connections:
- net N$98: now also TL1.3, TL2.3, TL3.3, TL4.3, TL5.3; no longer TL1.2, TL2.2, TL3.2, TL4.2, TL5.2
Routing:
- net N$98: track 75.1 -> 70.0 mm
Changed lines of the file:
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@@
 <grid distance="12.5" unitdist="mil" unit="mm" style="lines" multiple="1" display="yes" altdistance="0.025" altunitdist="inch" altunit="inch"/>
 <layers>
-<layer number="1" name="Top" color="4" fill="1" visible="no" active="yes"/>
+<layer number="1" name="Top" color="4" fill="1" visible="yes" active="yes"/>
 <layer number="2" name="Route2" color="1" fill="3" visible="no" active="yes"/>
 <layer number="3" name="Route3" color="4" fill="3" visible="no" active="yes"/>
@@
 <layer number="17" name="Pads" color="2" fill="1" visible="yes" active="yes"/>
 <layer number="18" name="Vias" color="2" fill="1" visible="yes" active="yes"/>
-<layer number="19" name="Unrouted" color="6" fill="1" visible="no" active="yes"/>
+<layer number="19" name="Unrouted" color="6" fill="1" visible="yes" active="yes"/>
 <layer number="20" name="Dimension" color="15" fill="1" visible="yes" active="yes"/>
-<layer number="21" name="tPlace" color="7" fill="1" visible="no" active="yes"/>
+<layer number="21" name="tPlace" color="7" fill="1" visible="yes" active="yes"/>
 <layer number="22" name="bPlace" color="7" fill="1" visible="yes" active="yes"/>
-<layer number="23" name="tOrigins" color="15" fill="1" visible="no" active="yes"/>
-<layer number="24" name="bOrigins" color="15" fill="1" visible="no" active="yes"/>
-<layer number="25" name="tNames" color="7" fill="1" visible="no" active="yes"/>
+<layer number="23" name="tOrigins" color="15" fill="1" visible="yes" active="yes"/>
+<layer number="24" name="bOrigins" color="15" fill="1" visible="yes" active="yes"/>
+<layer number="25" name="tNames" color="7" fill="1" visible="yes" active="yes"/>
 <layer number="26" name="bNames" color="7" fill="1" visible="yes" active="yes"/>
 <layer number="27" name="tValues" color="7" fill="1" visible="no" active="yes"/>
@@
 <signal name="N$98" class="3">
 <contactref element="D1" pad="A"/>
-<contactref element="TL5" pad="2"/>
-<contactref element="TL4" pad="2"/>
-<contactref element="TL3" pad="2"/>
-<contactref element="TL2" pad="2"/>
-<contactref element="TL1" pad="2"/>
-<wire x1="193.88" y1="71.755" x2="193.88" y2="71.55" width="0.4064" layer="1"/>
-<wire x1="193.88" y1="71.55" x2="195.58" y2="69.85" width="0.4064" layer="1"/>
-<wire x1="195.58" y1="69.85" x2="195.58" y2="64.77" width="0.4064" layer="1"/>
-<wire x1="195.58" y1="64.77" x2="197.8406" y2="62.5094" width="0.4064" layer="1"/>
-<wire x1="197.8406" y1="62.5094" x2="197.8406" y2="61.5188" width="0.4064" layer="1"/>
-<wire x1="197.8406" y1="61.5188" x2="197.8406" y2="60.6806" width="0.4064" layer="16"/>
-<wire x1="197.8406" y1="60.6806" x2="195.58" y2="58.42" width="0.4064" layer="16"/>
-<wire x1="195.58" y1="58.42" x2="195.58" y2="48.26" width="0.4064" layer="16"/>
-<wire x1="195.58" y1="48.26" x2="195.58" y2="34.925" width="0.4064" layer="16"/>
-<wire x1="195.58" y1="34.925" x2="195.58" y2="24.765" width="0.4064" layer="16"/>
-<wire x1="195.58" y1="24.765" x2="197.7644" y2="22.5806" width="0.4064" layer="16"/>
-<wire x1="197.7644" y1="22.5806" x2="197.7644" y2="21.59" width="0.4064" layer="16"/>
-<wire x1="197.7644" y1="21.59" x2="197.8406" y2="21.5138" width="0.4064" layer="16"/>
-<wire x1="197.8406" y1="34.8488" x2="195.6562" y2="34.8488" width="0.4064" layer="16"/>
-<wire x1="195.6562" y1="34.8488" x2="195.58" y2="34.925" width="0.4064" layer="16"/>
-<wire x1="197.8406" y1="48.1838" x2="195.6562" y2="48.1838" width="0.4064" layer="16"/>
-<wire x1="195.6562" y1="48.1838" x2="195.58" y2="48.26" width="0.4064" layer="16"/>
-<wire x1="197.8406" y1="21.5138" x2="197.8406" y2="20.5994" width="0.4064" layer="16"/>
-<wire x1="197.8406" y1="20.5994" x2="199.0725" y2="19.3675" width="0.4064" layer="16"/>
-<wire x1="199.0725" y1="19.3675" x2="210.5025" y2="19.3675" width="0.4064" layer="16"/>
-<wire x1="210.5025" y1="19.3675" x2="211.8106" y2="20.6756" width="0.4064" layer="16"/>
-<wire x1="211.8106" y1="20.6756" x2="211.8106" y2="21.5138" width="0.4064" layer="16"/>
+<contactref element="TL5" pad="3"/>
+<contactref element="TL4" pad="3"/>
+<contactref element="TL3" pad="3"/>
+<contactref element="TL2" pad="3"/>
+<contactref element="TL1" pad="3"/>
+<wire x1="193.3194" y1="28.0162" x2="193.3575" y2="27.305" width="0.4064" layer="16"/>
+<wire x1="193.3575" y1="27.305" x2="195.6181" y2="25.0444" width="0.4064" layer="16"/>
+<wire x1="195.6181" y1="25.0444" x2="195.6181" y2="20.5994" width="0.4064" layer="16"/>
+<wire x1="195.6181" y1="20.5994" x2="196.85" y2="19.3675" width="0.4064" layer="16"/>
+<wire x1="196.85" y1="19.3675" x2="201.295" y2="19.3675" width="0.4064" layer="16"/>
+<wire x1="201.295" y1="19.3675" x2="207.3275" y2="25.4" width="0.4064" layer="16"/>
+<wire x1="207.3275" y1="25.4" x2="207.3275" y2="27.94" width="0.4064" layer="16"/>
+<wire x1="207.3275" y1="27.94" x2="207.2894" y2="28.0162" width="0.4064" layer="16"/>
+<wire x1="193.3194" y1="28.0162" x2="193.3194" y2="41.3512" width="0.4064" layer="16"/>
+<wire x1="193.3194" y1="41.3512" x2="193.3194" y2="54.61" width="0.4064" layer="16"/>
+<wire x1="193.3194" y1="54.6862" x2="193.3194" y2="68.0212" width="0.4064" layer="16"/>
+<wire x1="193.88" y1="71.755" x2="193.3194" y2="71.755" width="0.4064" layer="1"/>
+<wire x1="193.3194" y1="71.755" x2="193.3194" y2="68.0212" width="0.4064" layer="1"/>
+<wire x1="193.3194" y1="54.6862" x2="193.3194" y2="54.61" width="0.4064" layer="16"/>
 </signal>
 <signal name="N$99" class="3">
